File: sellerie3000.sch (KiCad schematic (older format))
At the start: 19 parts, among them J1 USB_C_Receptacle, J2 Conn_01x04, J3 Conn_01x02, J4 Conn_01x02, U1 FT230XQ-R

Commit message: wow much update many unfinished
Parts:
- removed J2: Conn_01x04, Pin_Headers:Pin_Header_Straight_1x04_Pitch2.54mm, symbol Conn_01x04
- removed J3, J4: Conn_01x02, Pin_Headers:Pin_Header_Straight_1x02_Pitch2.54mm, symbol Conn_01x02
- removed JP1: VMODE, sellerie3000:Solder_Jumper, symbol Jumper_NO_Small
- added J2: Conn_01x05, Pin_Headers:Pin_Header_Straight_1x05_Pitch2.54mm, symbol Conn_01x05
- added TP1: RTS, Measurement_Points:Measurement_Point_Round-SMD-Pad_Small, symbol TEST
- added TP2: CTS, Measurement_Points:Measurement_Point_Round-SMD-Pad_Small, symbol TEST
- C1: renamed from C4; footprint Capacitors_SMD:C_0603 -> Capacitors_SMD:C_0402
- C2: footprint Capacitors_SMD:C_0603 -> Capacitors_SMD:C_0402
- C3: renamed from C1; footprint Capacitors_SMD:C_0603 -> Capacitors_SMD:C_0402
- C4: renamed from C3; footprint Capacitors_SMD:C_1206 -> Capacitors_SMD:C_0402
- C5: footprint Capacitors_SMD:C_1206 -> Capacitors_SMD:C_0402
- C6: footprint Capacitors_SMD:C_1206 -> Capacitors_SMD:C_0603
- J1: footprint Connectors_USB:USB_C_Receptacle_Amphenol_12401610E4-2A -> DX07B024JJ3:DX07B024JJ3
- R1, R2, R3, R4: footprint Resistors_SMD:R_0603 -> Resistors_SMD:R_0402
Connections:
- net VCCIO is gone; now on net 3V3: R3.1, R4.1, U1.1 (VCCIO)
- net 3V3: now also J2.2 (Pin_2)
- net CTS: now also TP2.1
- net GND: now also J2.5 (Pin_5)
- net RTS: now also TP1.1
- net RX: now also J2.3 (Pin_3)
- net TX: now also J2.4 (Pin_4)
- net VCC: now also L1.1, U1.10 (VCC), J2.1 (Pin_1); no longer C1.1, J1.A4 (VBUS), J1.A9 (VBUS), J1.B4 (VBUS), J1.B9 (VBUS), L1.2
- net USBDP: now reaches C3.1, R2.1, U1.6 (USBDP)
- net USBDM: now reaches C2.1, R1.1, U1.7 (USBDM)
- new net: C1.1, J1.A4 (VBUS), J1.A9 (VBUS), J1.B4 (VBUS), J1.B9 (VBUS), L1.2
Other:
- moved on the sheet: C5, C6, D1, D2, R3, R4
