File: darling.sch (KiCad schematic (older format))
At the start: 16 parts, among them J1 USB_C_Receptacle_USB2.0, J2 Conn_01x05, U1 FT230XQ

Commit message: fixed #4 usb-c is now reversable
Changed lines of the file:
@@
 EESchema Schematic File Version 4
-EELAYER 26 0
+LIBS:darling-cache
+EELAYER 29 0
 EELAYER END
 $Descr A4 11693 8268
@@
 $Comp
 L Connector_Generic:Conn_01x05 J2
-U 1 1 5C9AEA0C
+U 0 0 5C9AEA0C
 P 6750 4400
 F 0 "J2" H 6830 4442 50  0000 L CNN
@@
 F 2 "Connector_PinHeader_2.54mm:PinHeader_1x05_P2.54mm_Vertical" H 6750 4400 50  0001 C CNN
 F 3 "~" H 6750 4400 50  0001 C CNN
-	1    6750 4400
+	0    6750 4400
 	1    0    0    -1
 $EndComp
@@
 	6500 4150 6500 4200
 Wire Wire Line
-	6500 4200 6550 4200
-Wire Wire Line
 	6550 4300 6500 4300
 Wire Wire Line
@@
 NoConn ~ 3600 3600
 NoConn ~ 3600 3700
+Wire Wire Line
+	6500 4200 6550 4200
 $EndSCHEMATC
