File: darling.kicad_pcb (KiCad board)
At the start: 2 copper layers, 24 x 14 mm, 19 parts, among them J1 USB_C_Receptacle_USB2.0, J2 Conn_01x05, U1 FT230XQ

Commit message: final rev 4
Parts:
- removed the G*** at (102.2, 146.9)
- added G***: LOGO, 002:002_inv, B.Cu at (102.2, 146.9)
- added TP1: TestPoint, TestPoint:TestPoint_Pad_D1.0mm, F.Cu at (105.5, 142.0)
- added TP2: TestPoint, TestPoint:TestPoint_Pad_D1.0mm, F.Cu at (105.2, 154.0)
- moved C2 1.00 mm to (105.0, 144.0)
- moved C3 1.00 mm to (104.0, 144.0)
Routing:
- net /RTS: track 0.00 -> 16.8 mm
- net GND: track 37.3 -> 51.0 mm
- net /CTS: track 0.00 -> 12.9 mm, vias 0 -> 2
- net +3V3: track 25.3 -> 33.9 mm
- net VCC: track 16.1 -> 20.7 mm
Other:
- board text added: "CTS"
- board text added: "GND"
- board text added: "RTS"
- board text added: "darling.xengi.de v4"
- board text removed: "G"
- board text removed: "darling.xengi.de rev4"

Commit message: update readme and images
Parts:
- moved G*** 0.06 mm to (102.3, 146.9)
Changed lines of the file:
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@@
   )
   (footprint "002:002_inv" (layer "B.Cu")
-    (at 102.242869 146.89624 180)
+    (at 102.3 146.9 180)
     (attr board_only exclude_from_pos_files exclude_from_bom)
     (fp_text reference "G***" (at 0 0) (layer "B.SilkS") hide
