File: darling.kicad_sch (KiCad schematic)
At the start: 20 parts, among them J1 USB_C_Receptacle_USB2.0, J2 Conn_01x05, U1 FT230XQ

Commit message: add LCSC and Mouser part numbers
Parts:
- C1: LCSC (none) -> C272878; Mouser (none) -> 80-C0402C103K3R7867
- C2, C4: LCSC (none) -> C541464; Mouser (none) -> 81-GRM155C71H104JE9J
- C3: LCSC (none) -> C368809; Mouser (none) -> 81-GRM15C61E475ME15J
- C5, C6: LCSC (none) -> C527009; Mouser (none) -> 81-GRT1555C1H470FA2D
- D1: LCSC (none) -> C965804; Mouser (none) -> 710-150060GS75000
- D2: LCSC (none) -> C965799; Mouser (none) -> 710-150060RS75000
- FB1: LCSC (none) -> C21286; Mouser (none) -> 875-MI0805K601R-10
- J1: LCSC (none) -> C778726; Mouser (none) -> 798-CX70M-24P1
- J2: LCSC (none) -> C6332198; Mouser (none) -> 910-HDR100IMP40MGVTH
- R1, R2: LCSC (none) -> C138021; Mouser (none) -> 652-CR0402FX-27R0GLF
- R3, R4: LCSC (none) -> C163474; Mouser (none) -> 652-CR0402FX-2700GLF
- R5, R6: LCSC (none) -> C105873; Mouser (none) -> 652-CR0402FX-5101GLF
- U1: LCSC (none) -> C128629; Mouser (none) -> 895-FT230XQ-R
Changed lines of the file:
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@@
+      (effects (font (size 1.27 1.27)) hide)
+    )
+    (property "LCSC" "C128629" (at 127 82.55 0)
+      (effects (font (size 1.27 1.27)) hide)
+    )
+    (property "Mouser" "895-FT230XQ-R" (at 127 82.55 0)
       (effects (font (size 1.27 1.27)) hide)
     )
@@
       (effects (font (size 1.27 1.27)) hide)
     )
+    (property "LCSC" "C541464" (at 106.68 97.79 0)
+      (effects (font (size 1.27 1.27)) hide)
+    )
+    (property "Mouser" "81-GRM155C71H104JE9J" (at 106.68 97.79 0)
+      (effects (font (size 1.27 1.27)) hide)
+    )
     (pin "1")
     (pin "2")
@@
       (effects (font (size 1.27 1.27)) hide)
     )
+    (property "LCSC" "C541464" (at 69.85 109.22 0)
+      (effects (font (size 1.27 1.27)) hide)
+    )
+    (property "Mouser" "81-GRM155C71H104JE9J" (at 69.85 109.22 0)
+      (effects (font (size 1.27 1.27)) hide)
+    )
     (pin "1")
     (pin "2")
@@
       (effects (font (size 1.27 1.27)) hide)
     )
+    (property "LCSC" "C368809" (at 82.55 109.22 0)
+      (effects (font (size 1.27 1.27)) hide)
+    )
+    (property "Mouser" "81-GRM15C61E475ME15J" (at 82.55 109.22 0)
+      (effects (font (size 1.27 1.27)) hide)
+    )
     (pin "1")
     (pin "2")
@@
     )
     (property "Datasheet" "https://www.usb.org/sites/default/files/documents/usb_type-c.zip" (at 62.23 78.74 0)
+      (effects (font (size 1.27 1.27)) hide)
+    )
+    (property "LCSC" "C778726" (at 58.42 78.74 0)
+      (effects (font (size 1.27 1.27)) hide)
+    )
+    (property "Mouser" "798-CX70M-24P1" (at 58.42 78.74 0)
       (effects (font (size 1.27 1.27)) hide)
     )
@@
       (effects (font (size 1.27 1.27)) hide)
     )
+    (property "LCSC" "C21286" (at 96.52 63.5 0)
+      (effects (font (size 1.27 1.27)) hide)
+    )
+    (property "Mouser" "875-MI0805K601R-10" (at 96.52 63.5 0)
+      (effects (font (size 1.27 1.27)) hide)
+    )
     (pin "1")
     (pin "2")
@@
       (effects (font (size 1.27 1.27)) hide)
     )
+    (property "LCSC" "C138021" (at 100.33 82.55 0)
+      (effects (font (size 1.27 1.27)) hide)
+    )
+    (property "Mouser" "652-CR0402FX-27R0GLF" (at 100.33 82.55 0)
+      (effects (font (size 1.27 1.27)) hide)
+    )
     (pin "1")
     (pin "2")
@@
       (effects (font (size 1.27 1.27)) hide)
     )
+    (property "LCSC" "C138021" (at 92.71 80.01 0)
+      (effects (font (size 1.27 1.27)) hide)
+    )
+    (property "Mouser" "652-CR0402FX-27R0GLF" (at 92.71 80.01 0)
+      (effects (font (size 1.27 1.27)) hide)
+    )
     (pin "1")
     (pin "2")
@@
       (effects (font (size 1.27 1.27)) hide)
     )
+    (property "LCSC" "C527009" (at 90.17 87.63 0)
+      (effects (font (size 1.27 1.27)) hide)
+    )
+    (property "Mouser" "81-GRT1555C1H470FA2D" (at 90.17 87.63 0)
+      (effects (font (size 1.27 1.27)) hide)
+    )
     (pin "1")
     (pin "2")
@@
     )
     (property "Datasheet" "~" (at 77.47 87.63 0)
+      (effects (font (size 1.27 1.27)) hide)
+    )
+    (property "LCSC" "C527009" (at 77.47 87.63 0)
+      (effects (font (size 1.27 1.27)) hide)
+    )
+    (property "Mouser" "81-GRT1555C1H470FA2D" (at 77.47 87.63 0)
       (effects (font (size 1.27 1.27)) hide)
     )
@@
       (effects (font (size 1.27 1.27)) hide)
     )
+    (property "LCSC" "C965804" (at 154.94 71.12 0)
+      (effects (font (size 1.27 1.27)) hide)
+    )
+    (property "Mouser" "710-150060GS75000" (at 154.94 71.12 0)
+      (effects (font (size 1.27 1.27)) hide)
+    )
     (pin "1")
     (pin "2")
@@
       (effects (font (size 1.27 1.27)) hide)
     )
+    (property "LCSC" "C965799" (at 165.1 71.12 0)
+      (effects (font (size 1.27 1.27)) hide)
+    )
+    (property "Mouser" "710-150060RS75000" (at 165.1 71.12 0)
+      (effects (font (size 1.27 1.27)) hide)
+    )
     (pin "1")
     (pin "2")
@@
       (effects (font (size 1.27 1.27)) hide)
     )
+    (property "LCSC" "C163474" (at 154.94 80.01 0)
+      (effects (font (size 1.27 1.27)) hide)
+    )
+    (property "Mouser" "652-CR0402FX-2700GLF" (at 154.94 80.01 0)
+      (effects (font (size 1.27 1.27)) hide)
+    )
     (pin "1")
     (pin "2")
@@
       (effects (font (size 1.27 1.27)) hide)
     )
+    (property "LCSC" "C163474" (at 165.1 80.01 0)
+      (effects (font (size 1.27 1.27)) hide)
+    )
+    (property "Mouser" "652-CR0402FX-2700GLF" (at 165.1 80.01 0)
+      (effects (font (size 1.27 1.27)) hide)
+    )
     (pin "1")
     (pin "2")
@@
     )
     (property "Datasheet" "~" (at 156.21 109.22 0)
+      (effects (font (size 1.27 1.27)) hide)
+    )
+    (property "LCSC" "C6332198" (at 156.21 109.22 0)
+      (effects (font (size 1.27 1.27)) hide)
+    )
+    (property "Mouser" "910-HDR100IMP40MGVTH" (at 156.21 109.22 0)
       (effects (font (size 1.27 1.27)) hide)
     )
@@
       (effects (font (size 1.27 1.27)) hide)
     )
+    (property "LCSC" "" (at 119.38 110.49 0)
+      (effects (font (size 1.27 1.27)) hide)
+    )
+    (property "Mouser" "" (at 119.38 110.49 0)
+      (effects (font (size 1.27 1.27)) hide)
+    )
     (pin "1")
     (instances
@@
       (effects (font (size 1.27 1.27)) hide)
     )
+    (property "LCSC" "C105873" (at 77.47 68.58 0)
+      (effects (font (size 1.27 1.27)) hide)
+    )
+    (property "Mouser" "652-CR0402FX-5101GLF" (at 77.47 68.58 0)
+      (effects (font (size 1.27 1.27)) hide)
+    )
     (pin "1")
     (pin "2")
@@
     )
     (property "Datasheet" "~" (at 85.09 67.31 0)
+      (effects (font (size 1.27 1.27)) hide)
+    )
+    (property "LCSC" "C272878" (at 85.09 67.31 0)
+      (effects (font (size 1.27 1.27)) hide)
+    )
+    (property "Mouser" "80-C0402C103K3R7867" (at 85.09 67.31 0)
       (effects (font (size 1.27 1.27)) hide)
     )
@@
       (effects (font (size 1.27 1.27)) hide)
     )
+    (property "LCSC" "" (at 119.38 115.57 0)
+      (effects (font (size 1.27 1.27)) hide)
+    )
+    (property "Mouser" "" (at 119.38 115.57 0)
+      (effects (font (size 1.27 1.27)) hide)
+    )
     (pin "1")
     (instances
@@
       (effects (font (size 1.27 1.27)) hide)
     )
+    (property "LCSC" "C105873" (at 77.47 71.12 0)
+      (effects (font (size 1.27 1.27)) hide)
+    )
+    (property "Mouser" "652-CR0402FX-5101GLF" (at 77.47 71.12 0)
+      (effects (font (size 1.27 1.27)) hide)
+    )

Commit message: update pin header
Parts:
- J2: Mouser 910-HDR100IMP40MGVTH -> 571-826947-5
Changed lines of the file:
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@@
       (effects (font (size 1.27 1.27)) hide)
     )
-    (property "Mouser" "910-HDR100IMP40MGVTH" (at 156.21 109.22 0)
+    (property "Mouser" "571-826947-5" (at 156.21 109.22 0)
       (effects (font (size 1.27 1.27)) hide)
     )
